File: smartplug/smartplug.sch (KiCad schematic (older format))
At the start: 7 parts, among them U1 RAC01-05SGA, U2 RAC01-05SGA

Commit message: Added LED
Parts:
- added D?: LED, symbol Device:LED
- added R?: R, symbol Device:R
- K?: symbol ALA2F12:ALA2F12 -> smartplug-rescue:ALA2F12-ALA2F12
- U1, U2: symbol RAC01-05SGA:RAC01-05SGA -> smartplug-rescue:RAC01-05SGA-RAC01-05SGA
- U?: symbol particle-boards:PHOTON -> smartplug-rescue:PHOTON-particle-boards
- U?: symbol NUD3112LT1G:NUD3112LT1G -> smartplug-rescue:NUD3112LT1G-NUD3112LT1G
Connections:
- wire segments 22 -> 26
Changed lines of the file:
@@
 $EndDescr
 $Comp
-L particle-boards:PHOTON U?
+L smartplug-rescue:PHOTON-particle-boards U?
 U 1 1 5C931075
 P 5400 3350
@@
 $EndComp
 $Comp
-L NUD3112LT1G:NUD3112LT1G U?
+L smartplug-rescue:NUD3112LT1G-NUD3112LT1G U?
 U 1 1 5C931113
 P 7800 3250
@@
 $EndComp
 $Comp
-L RAC01-05SGA:RAC01-05SGA U1
+L smartplug-rescue:RAC01-05SGA-RAC01-05SGA U1
 U 1 1 5C9312A5
-P 2300 2700
-F 0 "U1" H 2300 3065 50  0000 C CNN
-F 1 "RAC01-05SGA" H 2300 2974 50  0000 C CNN
-F 2 "CONV_RAC01-05SGA" H 2300 2700 50  0001 L BNN
-F 3 "RAC01-05SGA" H 2300 2700 50  0001 L BNN
-F 4 "DIP-4 Recom Power" H 2300 2700 50  0001 L BNN "Field4"
-F 5 "Unavailable" H 2300 2700 50  0001 L BNN "Field5"
-F 6 "RAC01 Series Single Output 5 V 1 W POWERLINE AC/DC Converter" H 2300 2700 50  0001 L BNN "Field6"
-F 7 "Recom Power" H 2300 2700 50  0001 L BNN "Field7"
-F 8 "None" H 2300 2700 50  0001 L BNN "Field8"
-	1    2300 2700
-	1    0    0    -1
-$EndComp
-$Comp
-L RAC01-05SGA:RAC01-05SGA U2
+P 2250 1600
+F 0 "U1" H 2250 1965 50  0000 C CNN
+F 1 "RAC01-05SGA" H 2250 1874 50  0000 C CNN
+F 2 "CONV_RAC01-05SGA" H 2250 1600 50  0001 L BNN
+F 3 "RAC01-05SGA" H 2250 1600 50  0001 L BNN
+F 4 "DIP-4 Recom Power" H 2250 1600 50  0001 L BNN "Field4"
+F 5 "Unavailable" H 2250 1600 50  0001 L BNN "Field5"
+F 6 "RAC01 Series Single Output 5 V 1 W POWERLINE AC/DC Converter" H 2250 1600 50  0001 L BNN "Field6"
+F 7 "Recom Power" H 2250 1600 50  0001 L BNN "Field7"
+F 8 "None" H 2250 1600 50  0001 L BNN "Field8"
+	1    2250 1600
+	1    0    0    -1
+$EndComp
+$Comp
+L smartplug-rescue:RAC01-05SGA-RAC01-05SGA U2
 U 1 1 5C93137A
 P 2300 3450
@@
 12VDC
 $Comp
-L ALA2F12:ALA2F12 K?
+L smartplug-rescue:ALA2F12-ALA2F12 K?
 U 1 1 5C9402BB
 P 9050 2600
@@
 L power:GND #PWR?
 U 1 1 5C940AD6
-P 3000 2800
-F 0 "#PWR?" H 3000 2550 50  0001 C CNN
-F 1 "GND" H 3005 2627 50  0000 C CNN
-F 2 "" H 3000 2800 50  0001 C CNN
-F 3 "" H 3000 2800 50  0001 C CNN
-	1    3000 2800
-	1    0    0    -1
-$EndComp
-Wire Wire Line
-	3000 2600 3400 2600
+P 2950 1700
+F 0 "#PWR?" H 2950 1450 50  0001 C CNN
+F 1 "GND" H 2955 1527 50  0000 C CNN
+F 2 "" H 2950 1700 50  0001 C CNN
+F 3 "" H 2950 1700 50  0001 C CNN
+	1    2950 1700
+	1    0    0    -1
+$EndComp
+Wire Wire Line
+	2950 1500 3350 1500
 $Comp
 L power:+3V3 #PWR?
 U 1 1 5C940C6F
-P 3400 2600
-F 0 "#PWR?" H 3400 2450 50  0001 C CNN
-F 1 "+3V3" H 3415 2773 50  0000 C CNN
-F 2 "" H 3400 2600 50  0001 C CNN
-F 3 "" H 3400 2600 50  0001 C CNN
-	1    3400 2600
+P 3350 1500
+F 0 "#PWR?" H 3350 1350 50  0001 C CNN
+F 1 "+3V3" H 3365 1673 50  0000 C CNN
+F 2 "" H 3350 1500 50  0001 C CNN
+F 3 "" H 3350 1500 50  0001 C CNN
+	1    3350 1500
 	1    0    0    -1
 $EndComp
@@
 $EndComp
 Wire Wire Line
-	6200 3250 7100 3250
+	6200 3250 6650 3250
 Wire Wire Line
 	1100 2850 1300 2850
@@
 VAC-
 Wire Wire Line
-	1600 2600 1450 2600
-Wire Wire Line
-	1600 2800 1450 2800
+	1550 1500 1400 1500
+Wire Wire Line
+	1550 1700 1400 1700
 Wire Wire Line
 	1600 3350 1450 3350
 Wire Wire Line
 	1600 3550 1450 3550
-Text Label 1500 2600 0    50   ~ 0
-VAC+
-Text Label 1450 2800 0    50   ~ 0
+Text Label 1450 1500 0    50   ~ 0
+VAC+
+Text Label 1400 1700 0    50   ~ 0
 VAC-
 Text Label 1450 3350 0    50   ~ 0
@@
 Text Label 9450 3150 1    50   ~ 0
 VAC-
+$Comp
+L Device:LED D?
+U 1 1 5CA2FB4F
+P 6650 3900
+F 0 "D?" V 6688 3783 50  0000 R CNN
+F 1 "LED" V 6597 3783 50  0000 R CNN
+F 2 "" H 6650 3900 50  0001 C CNN
+F 3 "~" H 6650 3900 50  0001 C CNN
+	1    6650 3900
+	0    -1   -1   0
+$EndComp
+Wire Wire Line
+	6650 3250 6650 3750
+Connection ~ 6650 3250
+Wire Wire Line
+	6650 3250 7100 3250
+$Comp
+L Device:R R?
+U 1 1 5CA346F7
+P 6650 4400
+F 0 "R?" H 6720 4446 50  0000 L CNN
+F 1 "R" H 6720 4355 50  0000 L CNN
+F 2 "" V 6580 4400 50  0001 C CNN
+F 3 "~" H 6650 4400 50  0001 C CNN
+	1    6650 4400
+	1    0    0    -1
+$EndComp
+$Comp
+L power:GND #PWR?
+U 1 1 5CA34749
+P 6650 4650
+F 0 "#PWR?" H 6650 4400 50  0001 C CNN
+F 1 "GND" H 6655 4477 50  0000 C CNN
+F 2 "" H 6650 4650 50  0001 C CNN
+F 3 "" H 6650 4650 50  0001 C CNN
+	1    6650 4650
+	1    0    0    -1
+$EndComp
+Wire Wire Line
+	6650 4550 6650 4650
+Wire Wire Line
+	6650 4050 6650 4250
 $EndSCHEMATC

Commit message: Added schematic from usb charger
Parts:
- removed U1: RAC01-05SGA, CONV_RAC01-05SGA, symbol smartplug-rescue:RAC01-05SGA-RAC01-05SGA
- added C?: 10u, Capacitor_SMD:C_0805_2012Metric, symbol Device:C
- added C? (x2): 22u, Capacitor_SMD:C_0805_2012Metric, symbol Device:C
- added C?: 0.1u, Capacitor_SMD:C_0402_1005Metric, symbol Device:C
- added D?: D_Schottky, Diode_SMD:D_SMB, symbol Device:D_Schottky
- added L?: 6.8u, usb_charger:IND_SRR1240-6R8M, symbol Device:L
- added R?: 100k, Resistor_SMD:R_0402_1005Metric, symbol Device:R_US
- added U?: ADP2302ARDZ-5.0-R7, SOIC127P600X175-9N:SOIC127P600X175-9N, symbol usb_charger:ADP2302ARDZ-5.0-R7
- renumbered U2 to U?
Connections:
- net labels added: 5VDC
- net labels removed: +3V3
- wire segments 26 -> 39
- no-connect marks 0 -> 1
Other:
- moved on the sheet: D?, J?, K?, R?, U?

Commit message: added circuit protection
Parts:
- added RV?: Varistor, symbol Device:Varistor
Connections:
- wire segments 39 -> 43
Other:
- moved on the sheet: U?
Changed lines of the file:
@@
 EESchema Schematic File Version 4
 LIBS:smartplug-cache
-LIBS:USBCharger-cache
 EELAYER 26 0
 EELAYER END
@@
 L smartplug-rescue:RAC01-05SGA-RAC01-05SGA U?
 U 1 1 5C93137A
-P 2550 2400
-F 0 "U?" H 2550 2765 50  0000 C CNN
-F 1 "RAC01-05SGA" H 2550 2674 50  0000 C CNN
-F 2 "CONV_RAC01-05SGA" H 2550 2400 50  0001 L BNN
-F 3 "RAC01-05SGA" H 2550 2400 50  0001 L BNN
-F 4 "DIP-4 Recom Power" H 2550 2400 50  0001 L BNN "Field4"
-F 5 "Unavailable" H 2550 2400 50  0001 L BNN "Field5"
-F 6 "RAC01 Series Single Output 5 V 1 W POWERLINE AC/DC Converter" H 2550 2400 50  0001 L BNN "Field6"
-F 7 "Recom Power" H 2550 2400 50  0001 L BNN "Field7"
-F 8 "None" H 2550 2400 50  0001 L BNN "Field8"
-	1    2550 2400
+P 2400 2700
+F 0 "U?" H 2400 3065 50  0000 C CNN
+F 1 "RAC01-05SGA" H 2400 2974 50  0000 C CNN
+F 2 "CONV_RAC01-05SGA" H 2400 2700 50  0001 L BNN
+F 3 "RAC01-05SGA" H 2400 2700 50  0001 L BNN
+F 4 "DIP-4 Recom Power" H 2400 2700 50  0001 L BNN "Field4"
+F 5 "Unavailable" H 2400 2700 50  0001 L BNN "Field5"
+F 6 "RAC01 Series Single Output 5 V 1 W POWERLINE AC/DC Converter" H 2400 2700 50  0001 L BNN "Field6"
+F 7 "Recom Power" H 2400 2700 50  0001 L BNN "Field7"
+F 8 "None" H 2400 2700 50  0001 L BNN "Field8"
+	1    2400 2700
 	1    0    0    -1
 $EndComp
@@
 L power:GND #PWR0103
 U 1 1 5C940AA6
-P 3250 2500
-F 0 "#PWR0103" H 3250 2250 50  0001 C CNN
-F 1 "GND" H 3255 2327 50  0000 C CNN
-F 2 "" H 3250 2500 50  0001 C CNN
-F 3 "" H 3250 2500 50  0001 C CNN
-	1    3250 2500
-	1    0    0    -1
-$EndComp
-Wire Wire Line
-	3250 2300 3650 2300
-Text Label 3400 2300 0    50   ~ 0
+P 3100 2800
+F 0 "#PWR0103" H 3100 2550 50  0001 C CNN
+F 1 "GND" H 3105 2627 50  0000 C CNN
+F 2 "" H 3100 2800 50  0001 C CNN
+F 3 "" H 3100 2800 50  0001 C CNN
+	1    3100 2800
+	1    0    0    -1
+$EndComp
+Wire Wire Line
+	3100 2600 3500 2600
+Text Label 3250 2600 0    50   ~ 0
 12VDC
 $Comp
@@
 	6050 2800 6500 2800
 Wire Wire Line
-	1350 1800 1550 1800
-Wire Wire Line
 	1350 1900 1700 1900
 Wire Wire Line
@@
 VAC-
 Wire Wire Line
-	1850 2300 1700 2300
-Wire Wire Line
-	1850 2500 1700 2500
-Text Label 1700 2300 0    50   ~ 0
+	1700 2600 1550 2600
+Wire Wire Line
+	1700 2800 1550 2800
+Text Label 1550 2600 0    50   ~ 0
 VAC+
-Text Label 1700 2500 0    50   ~ 0
+Text Label 1550 2800 0    50   ~ 0
 VAC-
 $Comp
@@
 Text Label 4300 2200 0    50   ~ 0
 5VDC
+$Comp
+L Device:Varistor RV?
+U 1 1 5CA44C84
+P 2000 1900
+F 0 "RV?" H 2103 1946 50  0000 L CNN
+F 1 "Varistor" H 2103 1855 50  0000 L CNN
+F 2 "" V 1930 1900 50  0001 C CNN
+F 3 "~" H 2000 1900 50  0001 C CNN
+	1    2000 1900
+	1    0    0    -1
+$EndComp
+Wire Wire Line
+	1800 1800 1800 1750
+Wire Wire Line
+	1800 1750 2000 1750
+Wire Wire Line
+	1350 1800 1800 1800
+Wire Wire Line
+	1550 2000 1550 2050
+Wire Wire Line
+	1550 2050 2000 2050
 $EndSCHEMATC

Commit message: library fixes and female->male connector
Parts:
- removed J?: Conn_01x03_Female, symbol Connector:Conn_01x03_Female
- added J1: Conn_01x03_Male, symbol Connector:Conn_01x03_Male
- C2: renamed from C?; footprint Capacitor_SMD:C_0402_1005Metric -> Capacitor_SMD:C_0805_2012Metric
- D2: renamed from D?; footprint (none) -> LED_SMD:LED_0603_1608Metric
- U2: renamed from U?; symbol usb_charger:ADP2302ARDZ-5.0-R7 -> smartplug-rescue:ADP2302ARDZ-5.0-R7-usb_charger
- gave numbers to parts that had none: 13
Changed lines of the file:
@@
 $EndDescr
 $Comp
-L smartplug-rescue:PHOTON-particle-boards U?
+L smartplug-rescue:PHOTON-particle-boards U3
 U 1 1 5C931075
 P 5250 2900
-F 0 "U?" H 5250 3887 60  0000 C CNN
+F 0 "U3" H 5250 3887 60  0000 C CNN
 F 1 "PHOTON" H 5250 3781 60  0000 C CNN
-F 2 "" H 5250 3000 60  0000 C CNN
+F 2 "" H 5250 3000 60  0001 C CNN
 F 3 "" H 5250 3000 60  0000 C CNN
 	1    5250 2900
@@
 $EndComp
 $Comp
-L smartplug-rescue:NUD3112LT1G-NUD3112LT1G U?
+L smartplug-rescue:NUD3112LT1G-NUD3112LT1G U4
 U 1 1 5C931113
 P 7650 2800
-F 0 "U?" H 7650 3170 50  0000 C CNN
+F 0 "U4" H 7650 3170 50  0000 C CNN
 F 1 "NUD3112LT1G" H 7650 3079 50  0000 C CNN
 F 2 "SOT95P240X110-3N" H 7650 2800 50  0001 L BNN
@@
 $EndComp
 $Comp
-L Connector:Conn_01x03_Female J?
-U 1 1 5C931203
-P 1150 1900
-F 0 "J?" H 1044 1575 50  0000 C CNN
-F 1 "Conn_01x03_Female" H 1044 1666 50  0000 C CNN
-F 2 "" H 1150 1900 50  0001 C CNN
-F 3 "~" H 1150 1900 50  0001 C CNN
-	1    1150 1900
-	-1   0    0    1
-$EndComp
-$Comp
-L smartplug-rescue:RAC01-05SGA-RAC01-05SGA U?
+L smartplug-rescue:RAC01-05SGA-RAC01-05SGA U1
 U 1 1 5C93137A
 P 2400 2700
-F 0 "U?" H 2400 3065 50  0000 C CNN
+F 0 "U1" H 2400 3065 50  0000 C CNN
 F 1 "RAC01-05SGA" H 2400 2974 50  0000 C CNN
 F 2 "CONV_RAC01-05SGA" H 2400 2700 50  0001 L BNN
@@
 $EndComp
 $Comp
-L Connector:Conn_01x03_Female J?
+L Connector:Conn_01x03_Female J2
 U 1 1 5C93E3AE
 P 9900 1500
-F 0 "J?" H 9927 1526 50  0000 L CNN
+F 0 "J2" H 9927 1526 50  0000 L CNN
 F 1 "Conn_01x03_Female" H 9927 1435 50  0000 L CNN
 F 2 "" H 9900 1500 50  0001 C CNN
@@
 12VDC
 $Comp
-L smartplug-rescue:ALA2F12-ALA2F12 K?
+L smartplug-rescue:ALA2F12-ALA2F12 K1
 U 1 1 5C9402BB
 P 8900 2150
-F 0 "K?" H 9380 2196 50  0000 L CNN
+F 0 "K1" H 9380 2196 50  0000 L CNN
 F 1 "ALA2F12" H 9380 2105 50  0000 L CNN
 F 2 "Relay_THT:Relay_StandexMeder_DIP_LowProfile" H 9400 2100 50  0001 L CNN
@@
 VAC-
 $Comp
-L Device:LED D?
+L Device:LED D2
 U 1 1 5CA2FB4F
 P 6500 3450
-F 0 "D?" V 6538 3333 50  0000 R CNN
+F 0 "D2" V 6538 3333 50  0000 R CNN
 F 1 "LED" V 6447 3333 50  0000 R CNN
-F 2 "" H 6500 3450 50  0001 C CNN
+F 2 "LED_SMD:LED_0603_1608Metric" H 6500 3450 50  0001 C CNN
 F 3 "~" H 6500 3450 50  0001 C CNN
 	1    6500 3450
@@
 	6500 2800 6950 2800
 $Comp
-L Device:R R?
+L Device:R R2
 U 1 1 5CA346F7
 P 6500 3950
-F 0 "R?" H 6570 3996 50  0000 L CNN
+F 0 "R2" H 6570 3996 50  0000 L CNN
 F 1 "R" H 6570 3905 50  0000 L CNN
 F 2 "" V 6430 3950 50  0001 C CNN
@@
 	6500 3600 6500 3800
 $Comp
-L Device:C C?
+L Device:C C1
 U 1 1 5C6DDE21
 P 1450 6100
-F 0 "C?" H 1565 6146 50  0000 L CNN
+F 0 "C1" H 1565 6146 50  0000 L CNN
 F 1 "10u" H 1565 6055 50  0000 L CNN
 F 2 "Capacitor_SMD:C_0805_2012Metric" H 1488 5950 50  0001 C CNN
@@
 $EndComp
 $Comp
-L Device:C C?
+L Device:C C3
 U 1 1 5C6DDE69
 P 4200 5850
-F 0 "C?" H 4315 5896 50  0000 L CNN
+F 0 "C3" H 4315 5896 50  0000 L CNN
 F 1 "22u" H 4315 5805 50  0000 L CNN
 F 2 "Capacitor_SMD:C_0805_2012Metric" H 4238 5700 50  0001 C CNN
@@
 $EndComp
 $Comp
-L Device:C C?
+L Device:C C4
 U 1 1 5C6DDEB1
 P 4600 5850
-F 0 "C?" H 4715 5896 50  0000 L CNN
+F 0 "C4" H 4715 5896 50  0000 L CNN
 F 1 "22u" H 4715 5805 50  0000 L CNN
 F 2 "Capacitor_SMD:C_0805_2012Metric" H 4638 5700 50  0001 C CNN
@@
 $EndComp
 $Comp
-L Device:C C?
+L Device:C C2
 U 1 1 5C6DDF1F
 P 3300 5450
-F 0 "C?" H 3185 5404 50  0000 R CNN
+F 0 "C2" H 3185 5404 50  0000 R CNN
 F 1 "0.1u" H 3185 5495 50  0000 R CNN
-F 2 "Capacitor_SMD:C_0402_1005Metric" H 3338 5300 50  0001 C CNN
+F 2 "Capacitor_SMD:C_0805_2012Metric" H 3338 5300 50  0001 C CNN
 F 3 "~" H 3300 5450 50  0001 C CNN
 	1    3300 5450
@@
 $EndComp
 $Comp
-L usb_charger:ADP2302ARDZ-5.0-R7 U?
+L smartplug-rescue:ADP2302ARDZ-5.0-R7-usb_charger U2
 U 1 1 5C6DDC02
 P 2500 6050
-F 0 "U?" H 2500 6665 50  0000 C CNN
+F 0 "U2" H 2500 6665 50  0000 C CNN
 F 1 "ADP2302ARDZ-5.0-R7" H 2500 6574 50  0000 C CNN
 F 2 "SOIC127P600X175-9N:SOIC127P600X175-9N" H 2500 6650 50  0001 C CNN
@@
 Connection ~ 4600 5700
 $Comp
-L Device:L L?
+L Device:L L1
 U 1 1 5C6DE73A
 P 3750 5700
-F 0 "L?" V 3572 5700 50  0000 C CNN
+F 0 "L1" V 3572 5700 50  0000 C CNN
 F 1 "6.8u" V 3663 5700 50  0000 C CNN
 F 2 "usb_charger:IND_SRR1240-6R8M" H 3750 5700 50  0001 C CNN
@@
 $EndComp
 $Comp
-L Device:D_Schottky D?
+L Device:D_Schottky D1
 U 1 1 5C6DE7EA
 P 3300 5850
-F 0 "D?" V 3254 5929 50  0000 L CNN
+F 0 "D1" V 3254 5929 50  0000 L CNN
 F 1 "D_Schottky" V 3345 5929 50  0000 L CNN
 F 2 "Diode_SMD:D_SMB" H 3300 5850 50  0001 C CNN
@@
 	2050 5950 2050 6200
 $Comp
-L Device:R_US R?
+L Device:R_US R1
 U 1 1 5C6DEF30
 P 1800 6350
-F 0 "R?" H 1868 6396 50  0000 L CNN
+F 0 "R1" H 1868 6396 50  0000 L CNN
 F 1 "100k" H 1868 6305 50  0000 L CNN
 F 2 "Resistor_SMD:R_0402_1005Metric" V 1840 6340 50  0001 C CNN
@@
 5VDC
 $Comp
-L Device:Varistor RV?
+L Device:Varistor RV1
 U 1 1 5CA44C84
 P 2000 1900
-F 0 "RV?" H 2103 1946 50  0000 L CNN
+F 0 "RV1" H 2103 1946 50  0000 L CNN
 F 1 "Varistor" H 2103 1855 50  0000 L CNN
 F 2 "" V 1930 1900 50  0001 C CNN
@@
 Wire Wire Line
 	1550 2050 2000 2050
+$Comp
+L Connector:Conn_01x03_Male J1
+U 1 1 5CA5498D
+P 1150 1900
+F 0 "J1" H 1256 2178 50  0000 C CNN
+F 1 "Conn_01x03_Male" H 1256 2087 50  0000 C CNN
+F 2 "" H 1150 1900 50  0001 C CNN
+F 3 "~" H 1150 1900 50  0001 C CNN
+	1    1150 1900
+	1    0    0    -1
+$EndComp
 $EndSCHEMATC

Commit message: fix footprint libs
Parts:
- R2: footprint (none) -> Resistor_SMD:R_0805_2012Metric
- U1: footprint CONV_RAC01-05SGA -> RAC01-05SGA:CONV_RAC01-05SGA
- U3: footprint (none) -> digikey-footprints:Particle_Photon
- U4: footprint SOT95P240X110-3N -> NUD3112LT1G:SOT95P240X110-3N
Changed lines of the file:
@@
 F 0 "U3" H 5250 3887 60  0000 C CNN
 F 1 "PHOTON" H 5250 3781 60  0000 C CNN
-F 2 "" H 5250 3000 60  0001 C CNN
+F 2 "digikey-footprints:Particle_Photon" H 5250 3000 60  0001 C CNN
 F 3 "" H 5250 3000 60  0000 C CNN
 	1    5250 2900
@@
 F 0 "U4" H 7650 3170 50  0000 C CNN
 F 1 "NUD3112LT1G" H 7650 3079 50  0000 C CNN
-F 2 "SOT95P240X110-3N" H 7650 2800 50  0001 L BNN
+F 2 "NUD3112LT1G:SOT95P240X110-3N" H 7650 2800 50  0001 L BNN
 F 3 "NUD3112LT1GOSCT-ND" H 7650 2800 50  0001 L BNN
 F 4 "SOT-23-3 ON Semiconductor" H 7650 2800 50  0001 L BNN "Field4"
@@
 F 0 "U1" H 2400 3065 50  0000 C CNN
 F 1 "RAC01-05SGA" H 2400 2974 50  0000 C CNN
-F 2 "CONV_RAC01-05SGA" H 2400 2700 50  0001 L BNN
+F 2 "RAC01-05SGA:CONV_RAC01-05SGA" H 2400 2700 50  0001 L BNN
 F 3 "RAC01-05SGA" H 2400 2700 50  0001 L BNN
 F 4 "DIP-4 Recom Power" H 2400 2700 50  0001 L BNN "Field4"
@@
 F 0 "R2" H 6570 3996 50  0000 L CNN
 F 1 "R" H 6570 3905 50  0000 L CNN
-F 2 "" V 6430 3950 50  0001 C CNN
+F 2 "Resistor_SMD:R_0805_2012Metric" V 6430 3950 50  0001 C CNN
 F 3 "~" H 6500 3950 50  0001 C CNN
 	1    6500 3950

Commit message: assign footprints and netlist
Parts:
- J1, J2: footprint (none) -> female_plug:TE_3-213598-2
- RV1: footprint (none) -> FUSE_0154004.DR:FUSE_0154004.DR
Changed lines of the file:
@@
 F 0 "J2" H 9927 1526 50  0000 L CNN
 F 1 "Conn_01x03_Female" H 9927 1435 50  0000 L CNN
-F 2 "" H 9900 1500 50  0001 C CNN
+F 2 "female_plug:TE_3-213598-2" H 9900 1500 50  0001 C CNN
 F 3 "~" H 9900 1500 50  0001 C CNN
 	1    9900 1500
@@
 F 0 "RV1" H 2103 1946 50  0000 L CNN
 F 1 "Varistor" H 2103 1855 50  0000 L CNN
-F 2 "" V 1930 1900 50  0001 C CNN
+F 2 "FUSE_0154004.DR:FUSE_0154004.DR" V 1930 1900 50  0001 C CNN
 F 3 "~" H 2000 1900 50  0001 C CNN
 	1    2000 1900
@@
 F 0 "J1" H 1256 2178 50  0000 C CNN
 F 1 "Conn_01x03_Male" H 1256 2087 50  0000 C CNN
-F 2 "" H 1150 1900 50  0001 C CNN
+F 2 "female_plug:TE_3-213598-2" H 1150 1900 50  0001 C CNN
 F 3 "~" H 1150 1900 50  0001 C CNN
 	1    1150 1900

Commit message: change relay footprint
Parts:
- K1: footprint Relay_THT:Relay_StandexMeder_DIP_LowProfile -> ALA2F12_changed:ALA2F12-pins_changed
Changed lines of the file:
@@
 F 0 "K1" H 9380 2196 50  0000 L CNN
 F 1 "ALA2F12" H 9380 2105 50  0000 L CNN
-F 2 "Relay_THT:Relay_StandexMeder_DIP_LowProfile" H 9400 2100 50  0001 L CNN
+F 2 "ALA2F12_changed:ALA2F12-pins_changed" H 9400 2100 50  0001 L CNN
 F 3 "https://standexelectronics.com/wp-content/uploads/datasheet_reed_relay_DIP.pdf" H 8800 2150 50  0001 C CNN
 	1    8900 2150

Commit message: first draft layout
Parts:
- J1, J2: footprint female_plug:TE_3-213598-2 -> female_plug_new:TE_3-213598-2-new
Changed lines of the file:
@@
 F 0 "J2" H 9927 1526 50  0000 L CNN
 F 1 "Conn_01x03_Female" H 9927 1435 50  0000 L CNN
-F 2 "female_plug:TE_3-213598-2" H 9900 1500 50  0001 C CNN
+F 2 "female_plug_new:TE_3-213598-2-new" H 9900 1500 50  0001 C CNN
 F 3 "~" H 9900 1500 50  0001 C CNN
 	1    9900 1500
@@
 F 0 "J1" H 1256 2178 50  0000 C CNN
 F 1 "Conn_01x03_Male" H 1256 2087 50  0000 C CNN
-F 2 "female_plug:TE_3-213598-2" H 1150 1900 50  0001 C CNN
+F 2 "female_plug_new:TE_3-213598-2-new" H 1150 1900 50  0001 C CNN
 F 3 "~" H 1150 1900 50  0001 C CNN
 	1    1150 1900
